Commit message: feat(urdf): complete base structure with wheels and updated meshes

File: bin_description/urdf/bin_robot.urdf.xacro (robot description, xacro)
@@ -7,4 +7,5 @@
     <xacro:arg name="use_gazebo" default="true"/>
     <xacro:include filename="$(find bin_description)/urdf/body/bin_base.urdf.xacro"/>
+    <xacro:include filename="$(find bin_description)/urdf/body/bin_wheels.urdf.xacro"/>
     <!-- <xacro:include filename="$(find bin_description)/urdf/sensors/lidar.urdf.xacro"/>
     <xacro:include filename="$(find bin_description)/urdf/body/bin_wheel.urdf.xacro"/>
@@ -18,4 +19,8 @@
     prefix="$(arg prefix)"
     z_off="${wheel_radius}"/>  <!--Wheel Radius-->
+    <xacro:bin_motors
+      prefix="$(arg prefix)"/>
+    <xacro:bin_wheels
+      prefix="$(arg prefix)" />
     <!-- <xacro:back_bin_stud
       prefix="$(arg prefix)"

File: bin_description/urdf/body/bin_base.urdf.xacro (robot description, xacro)
@@ -24,8 +24,8 @@
                 <box size="${base_length} ${base_width} ${base_height}"/>
             </geometry>
-            <origin xyz="0 0 0" rpy="0 0 0"/>
+            <origin xyz="0 0 ${base_height - wheel_radius}" rpy="0 0 0"/>
         </collision>
         <inertial>
-            <origin xyz="${com_x} ${com_y} ${com_z}" rpy="0 0 0"/>
+            <origin xyz="0 0 0" rpy="0 0 0"/>
             <mass value="${base_mass}"/>
             <inertia ixx="${(1/12) * base_mass * ((base_width * base_width) + (base_height * base_height))}"  ixy="0.0"  ixz="0.0"
@@ -40,9 +40,4 @@
   </joint>
   <link name="bin_castor_link">
-    <inertial>
-        <origin xyz="0.0 0.0 0.0" rpy="0.0 0.0 0.0"/>
-        <mass value="0.0"/>
-        <inertia ixx="0.0" ixy="0.0" ixz="0.0" iyy="0.0" iyz="0.0" izz="0.0"/>
-    </inertial>
     <visual>
         <origin xyz="0.08 0.0 0.0" rpy="0.0 0.0 0.0"/>
@@ -56,9 +51,16 @@
     </visual>
     <collision>
-        <origin xyz="0.0 0.0 0.0" rpy="0.0 0.0 0.0"/>
+        <origin xyz="0.08 0.0 0.0" rpy="0.0 0.0 0.0"/>
         <geometry>
             <mesh filename="package://bin_description/meshes/Caster Wheel.stl" scale="1 1 1"/>
         </geometry>
     </collision>
+    <inertial>
+        <mass value="0.01"/>
+        <origin xyz="0.0 0.0 0.0" rpy="0.0 0.0 0.0"/>
+        <inertia ixx="0.0"  ixy="0.0"  ixz="0.0"
+                    iyy="3.288427e-6"  iyz="0.0"
+                    izz="3.29244e-6"/>
+    </inertial>
   </link>
   <joint name="base_castor_joint" type="fixed">

Commit message: feat(sim): add gazebo simulation, controllers, sensors, and SLAM integration (no Nav2)

File: bin_description/urdf/bin_robot.urdf.xacro (robot description, xacro)
@@ -10,4 +10,8 @@
     <xacro:include filename="$(find bin_description)/urdf/body/bin_top.urdf.xacro"/>
     <xacro:include filename="$(find bin_description)/urdf/body/bin_cover.urdf.xacro"/>
+    <xacro:include filename="$(find bin_description)/urdf/sensors/bin_camera.urdf.xacro"/>
+    <xacro:include filename="$(find bin_description)/urdf/sensors/bin_lidar.urdf.xacro"/>
+    <xacro:include filename="$(find bin_description)/urdf/ros2_control/bin_ros2_control.xacro"/>
+    <xacro:include filename="$(find bin_description)/urdf/gazebo/bin_gazebo.urdf.xacro"/>
     <!-- <xacro:include filename="$(find bin_description)/urdf/sensors/lidar.urdf.xacro"/>
     <xacro:include filename="$(find bin_description)/urdf/body/bin_wheel.urdf.xacro"/>
@@ -18,4 +22,6 @@
     <!-- <xacro:include filename="$(find bin_description)/urdf/sensors/rgbd_camera.urdf.xacro"/>
     <xacro:include filename="$(find bin_description)/urdf/sensors/imu.urdf.xacro"/> -->
+    <xacro:bin_ros2_control prefix="$(arg prefix)" use_gazebo="$(arg use_gazebo)" />
+    <xacro:bin_gazebo prefix="$(arg prefix)" />
     <xacro:bin_base
     prefix="$(arg prefix)"
@@ -29,4 +35,8 @@
       height="${base_height - wheel_radius}" />
     <xacro:bin_cover
+      prefix="$(arg prefix)" />
+    <xacro:bin_camera
+      prefix="$(arg prefix)" />
+    <xacro:bin_lidar
       prefix="$(arg prefix)" />
     <!-- <xacro:back_bin_stud

File: bin_description/urdf/body/bin_base.urdf.xacro (robot description, xacro)
@@ -22,5 +22,5 @@
         <collision>
             <geometry>
-                <box size="${base_length} ${base_width} ${base_height}"/>
+                <mesh filename="package://bin_description/meshes/Base.stl" scale="1 1 1"/>
             </geometry>
             <origin xyz="0 0 ${base_height - wheel_radius}" rpy="0 0 0"/>
@@ -39,5 +39,5 @@
         <origin xyz="0 0 ${z_off}" rpy="0 0 0"/>
   </joint>
-  <link name="bin_castor_link">
+  <link name="${prefix}bin_castor_link">
     <visual>
         <origin xyz="0.08 0.0 0.0" rpy="0.0 0.0 0.0"/>
@@ -64,8 +64,8 @@
     </inertial>
   </link>
-  <joint name="base_castor_joint" type="fixed">
+  <joint name="${prefix}base_castor_joint" type="fixed">
     <origin xyz="-0.08 0.0 0.0" rpy="0.0 0.0 0.0"/>
-    <parent link="base_link"/>
-    <child link="bin_castor_link"/>
+    <parent link="${prefix}base_link"/>
+    <child link="${prefix}bin_castor_link"/>
   </joint>
 </xacro:macro>

File: bin_description/urdf/body/bin_cover.urdf.xacro (robot description, xacro)
@@ -18,7 +18,7 @@
             <collision>
                 <geometry>
-                    <box size="${cover_length} ${cover_width} ${cover_height}"/>
+                    <mesh filename="package://bin_description/meshes/Cover.stl" scale="1 1 1"/>
                 </geometry>
-                <origin xyz="0 0 0" rpy="0 0 0"/>
+                <origin xyz="${cover_length/2} 0 ${-bin_height}" rpy="0 0 0"/>
             </collision>
             <inertial>

File: bin_description/urdf/body/bin_top.urdf.xacro (robot description, xacro)
@@ -18,5 +18,5 @@
             <collision>
                 <geometry>
-                    <box size="0.036 0.036 0.0768"/>
+                    <mesh filename="package://bin_description/meshes/Bin.stl" scale="1 1 1"/>
                 </geometry>
                 <origin xyz="0 0 0" rpy="0 0 0"/>

File: bin_description/urdf/body/bin_wheels.urdf.xacro (robot description, xacro)
@@ -18,7 +18,7 @@
             <collision>
                 <geometry>
-                    <box size="0.036 0.036 0.0768"/>
+                    <mesh filename="package://bin_description/meshes/Left Motor.stl" scale="1 1 1"/>
                 </geometry>
-                <origin xyz="0 -0.03 0" rpy="${pi/2} 0 ${pi/2}"/>
+                <origin xyz="0 0.03 0" rpy="${pi/2} 0 ${-pi/2}"/>
             </collision>
             <inertial>
@@ -48,5 +48,5 @@
             <collision>
                 <geometry>
-                    <box size="0.036 0.036 0.0768"/>
+                    <mesh filename="package://bin_description/meshes/Left Motor.stl" scale="1 1 1"/>
                 </geometry>
                 <origin xyz="0 -0.03 0" rpy="${pi/2} 0 ${pi/2}"/>
@@ -80,5 +80,5 @@
             <collision>
                 <geometry>
-                    <cylinder radius="${wheel_radius}" length="${wheel_width}"/>
+                    <mesh filename="package://bin_description/meshes/Left Wheel.stl" scale="1 1 1"/>
                 </geometry>
                 <origin xyz="0 0 0" rpy="0 0 ${pi}"/>
@@ -111,7 +111,7 @@
             <collision>
                 <geometry>
-                    <cylinder radius="${wheel_radius}" length="${wheel_width}"/>
+                    <mesh filename="package://bin_description/meshes/Right Wheel.stl" scale="1 1 1"/>
                 </geometry>
-                <origin xyz="0 0 0" rpy="0 0 ${pi}"/>
+                <origin xyz="0 0 0" rpy="0 0 0"/>
             </collision>
             <inertial>
