Commit message: feat: Add new world and navigation capabilities

File: bin_description/urdf/bin_robot.urdf.xacro (robot description, xacro)
@@ -26,18 +26,19 @@
     <xacro:bin_base
     prefix="$(arg prefix)"
-    z_off="${wheel_radius}"/>  <!--Wheel Radius-->
-    <xacro:bin_motors
+    z_off="${wheel_radius}"/>  <!--wheel_radius + motor z-offset (0.01) to land wheels on ground-->
+    <xacro:bin_wheels
       prefix="$(arg prefix)"/>
-    <xacro:bin_wheels
-      prefix="$(arg prefix)" />
     <xacro:bin_top
       prefix="$(arg prefix)"
-      height="${base_height - wheel_radius}" />
+      height="${base_height}" />
     <xacro:bin_cover
+      prefix="$(arg prefix)" />
+    <xacro:bin_lidar
       prefix="$(arg prefix)" />
     <xacro:bin_camera
       prefix="$(arg prefix)" />
-    <xacro:bin_lidar
-      prefix="$(arg prefix)" />
+    <!-- <xacro:bin_motors
+      prefix="$(arg prefix)"/>
+ -->
     <!-- <xacro:back_bin_stud
       prefix="$(arg prefix)"

File: bin_description/urdf/body/bin_base.urdf.xacro (robot description, xacro)
@@ -7,5 +7,10 @@
 <xacro:property name="com_y" value="-0.00007433" />
 <xacro:property name="com_z" value="0.001" />
-<xacro:property name="base_mass" value="1.5" />
+<xacro:property name="pla_density"        value="1240.0" />
+<xacro:property name="metal_density"      value="7850.0" />
+<xacro:property name="base_wall_thickness" value="0.004" />
+<xacro:property name="base_mass" value="${pla_density * base_wall_thickness * (base_length*base_width + 2*base_width*base_height + 2*base_length*base_height)}" />
+<xacro:property name="castor_radius" value="${wheel_radius/2}" />
+<xacro:property name="castor_mass" value="${metal_density * (4.0/3.0) * pi * castor_radius * castor_radius * castor_radius}" />
 <xacro:macro name="bin_base" params="prefix z_off">
     <link name="base_footprint"/>
@@ -13,7 +18,8 @@
         <visual>
             <geometry>
-                <mesh filename="package://bin_description/meshes/Base.stl" scale="1 1 1"/>
+                <!-- <mesh filename="package://bin_description/meshes/Base.stl" scale="1 1 1"/> -->
+                <box size="${base_length} ${base_width} ${base_height}"/>
             </geometry>
-            <origin xyz="0 0 ${base_height - wheel_radius}" rpy="0 0 0"/>
+            <origin xyz="0 0 ${base_height/2}" rpy="0 0 0"/>
             <material name="white">
                 <color rgba="1 1 1 0.5"/>
@@ -22,7 +28,8 @@
         <collision>
             <geometry>
-                <mesh filename="package://bin_description/meshes/Base.stl" scale="1 1 1"/>
+                <!-- <mesh filename="package://bin_description/meshes/Base.stl" scale="1 1 1"/> -->
+                <box size="${base_length} ${base_width} ${base_height}"/>
             </geometry>
-            <origin xyz="0 0 ${base_height - wheel_radius}" rpy="0 0 0"/>
+            <origin xyz="0 0 ${base_height/2}" rpy="0 0 0"/>
         </collision>
         <inertial>
@@ -38,35 +45,36 @@
         <child link="${prefix}base_link"/>
         <origin xyz="0 0 ${z_off}" rpy="0 0 0"/>
-  </joint>
-  <link name="${prefix}bin_castor_link">
-    <visual>
-        <origin xyz="0.08 0.0 0.0" rpy="0.0 0.0 0.0"/>
-        <!-- <origin xyz="0.0 0.0 0.011" rpy="0.0 0.0 0.0"/> -->
-        <geometry>
-            <mesh filename="package://bin_description/meshes/Caster Wheel.stl" scale="1 1 1"/>
-        </geometry>
-        <material name="black">
-            <color rgba="0 0 0 0.5"/>
-        </material>
-    </visual>
-    <collision>
-        <origin xyz="0.08 0.0 0.0" rpy="0.0 0.0 0.0"/>
-        <geometry>
-            <mesh filename="package://bin_description/meshes/Caster Wheel.stl" scale="1 1 1"/>
-        </geometry>
-    </collision>
-    <inertial>
-        <mass value="0.01"/>
-        <origin xyz="0.0 0.0 0.0" rpy="0.0 0.0 0.0"/>
-        <inertia ixx="0.0"  ixy="0.0"  ixz="0.0"
-                    iyy="3.288427e-6"  iyz="0.0"
-                    izz="3.29244e-6"/>
-    </inertial>
-  </link>
-  <joint name="${prefix}base_castor_joint" type="fixed">
-    <origin xyz="-0.08 0.0 0.0" rpy="0.0 0.0 0.0"/>
-    <parent link="${prefix}base_link"/>
-    <child link="${prefix}bin_castor_link"/>
-  </joint>
+    </joint>
+    <link name="${prefix}bin_castor_link">
+        <visual>
+            <origin xyz="0.0 0.0 0.0" rpy="0.0 0.0 0.0"/>
+            <geometry>
+                <!-- <mesh filename="package://bin_description/meshes/Caster Wheel.stl" scale="1 1 1"/> -->
+                <sphere radius="${castor_radius}"/>
+            </geometry>
+            <material name="black">
+                <color rgba="0 0 0 0.5"/>
+            </material>
+        </visual>
+        <collision>
+            <origin xyz="0.0 0.0 0.0" rpy="0.0 0.0 0.0"/>
+            <geometry>
+                <!-- <mesh filename="package://bin_description/meshes/Caster Wheel.stl" scale="1 1 1"/> -->
+                <sphere radius="${castor_radius}"/>
+            </geometry>
+        </collision>
+        <inertial>
+            <mass value="${castor_mass}"/>
+            <origin xyz="0.0 0.0 0.0" rpy="0.0 0.0 0.0"/>
+            <inertia ixx="${(2/5) * castor_mass * castor_radius * castor_radius}"  ixy="0.0"  ixz="0.0"
+                    iyy="${(2/5) * castor_mass * castor_radius * castor_radius}"  iyz="0.0"
+                    izz="${(2/5) * castor_mass * castor_radius * castor_radius}"/>
+        </inertial>
+    </link>
+    <joint name="${prefix}base_castor_joint" type="fixed">
+        <origin xyz="${-base_length/2} 0.0 ${-castor_radius}" rpy="0.0 0.0 0.0"/>
+        <parent link="${prefix}base_link"/>
+        <child link="${prefix}bin_castor_link"/>
+    </joint>
 </xacro:macro>
 </robot>

File: bin_description/urdf/body/bin_cover.urdf.xacro (robot description, xacro)
@@ -1,15 +1,17 @@
 <?xml version="1.0"?>
 <robot xmlns:xacro="http://www.ros.org/wiki/xacro">
-    <xacro:property name="cover_mass" value="0.18525" />
-    <xacro:property name="cover_length" value="0.266" />
-    <xacro:property name="cover_width" value="0.266" />
+    <xacro:property name="plastic_density" value="1050.0" />
+    <xacro:property name="cover_length" value="0.2" />
+    <xacro:property name="cover_width" value="0.2" />
     <xacro:property name="cover_height" value="0.012" />
+    <xacro:property name="cover_mass" value="${plastic_density * cover_length * cover_width * cover_height}" />
     <xacro:macro name="bin_cover" params="prefix">
         <link name="${prefix}bin_cover_link">
             <visual>
                 <geometry>
-                    <mesh filename="package://bin_description/meshes/Cover.stl" scale="1 1 1"/>
+                    <!-- <mesh filename="package://bin_description/meshes/Cover.stl" scale="1 1 1"/> -->
+                    <box size="${cover_length} ${cover_width} ${cover_height}"/>
                 </geometry>
-                <origin xyz="${cover_length/2} 0 ${-bin_height}" rpy="0 0 0"/>
+                <origin xyz="0.0 0.0 0.0" rpy="0 0 0"/>
                 <material name="black">
                     <color rgba="0 0 0 1"/>
@@ -18,7 +20,8 @@
             <collision>
                 <geometry>
-                    <mesh filename="package://bin_description/meshes/Cover.stl" scale="1 1 1"/>
+                    <!-- <mesh filename="package://bin_description/meshes/Cover.stl" scale="1 1 1"/> -->
+                    <box size="${cover_length} ${cover_width} ${cover_height}"/>
                 </geometry>
-                <origin xyz="${cover_length/2} 0 ${-bin_height}" rpy="0 0 0"/>
+                <origin xyz="0 0 0" rpy="0 0 0"/>
             </collision>
             <inertial>
@@ -33,5 +36,5 @@
             <parent link="${prefix}bin_top_link"/>
             <child link="${prefix}bin_cover_link"/>
-            <origin xyz="${-cover_length/2} 0 ${bin_height}" rpy="0 0 0"/>
+            <origin xyz="0 0 ${bin_height}" rpy="0 0 0"/>
             <axis xyz="0 1 0"/>
             <limit lower="${-pi/2}" upper="0" effort="10" velocity="1.0"/>

File: bin_description/urdf/body/bin_top.urdf.xacro (robot description, xacro)
@@ -1,15 +1,19 @@
 <?xml version="1.0"?>
 <robot xmlns:xacro="http://www.ros.org/wiki/xacro">
+    <xacro:property name="plastic_density"    value="1050.0" />
+    <xacro:property name="bin_wall_thickness" value="0.004"  />
+    <xacro:property name="bin_length" value="0.20" />
+    <xacro:property name="bin_width" value="0.20" />
+    <xacro:property name="bin_height" value="0.24" />
+    <!-- <xacro:property name="bin_mass" value="${plastic_density * bin_wall_thickness * (bin_length*bin_width + 2*bin_width*bin_height + 2*bin_length*bin_height)}" /> -->
     <xacro:property name="bin_mass" value="0.1" />
-    <xacro:property name="bin_length" value="0.270" />
-    <xacro:property name="bin_width" value="0.270" />
-    <xacro:property name="bin_height" value="0.3048" />
     <xacro:macro name="bin_top" params="prefix height">
         <link name="${prefix}bin_top_link">
             <visual>
                 <geometry>
-                    <mesh filename="package://bin_description/meshes/Bin.stl" scale="1 1 1"/>
+                    <!-- <mesh filename="package://bin_description/meshes/Bin.stl" scale="1 1 1"/> -->
+                    <box size="${bin_length} ${bin_width} ${bin_height}"/>
                 </geometry>
-                <origin xyz="0 0 0" rpy="0 0 0"/>
+                <origin xyz="0 0 ${bin_height/2}" rpy="0 0 0"/>
                 <material name="white">
                     <color rgba="1 1 1 1"/>
@@ -18,7 +22,8 @@
             <collision>
                 <geometry>
-                    <mesh filename="package://bin_description/meshes/Bin.stl" scale="1 1 1"/>
+                    <!-- <mesh filename="package://bin_description/meshes/Bin.stl" scale="1 1 1"/> -->
+                    <box size="${bin_length} ${bin_width} ${bin_height}"/>
                 </geometry>
-                <origin xyz="0 0 0" rpy="0 0 0"/>
+                <origin xyz="0 0 ${bin_height/2}" rpy="0 0 0"/>
             </collision>
             <inertial>

File: bin_description/urdf/body/bin_wheels.urdf.xacro (robot description, xacro)
@@ -1,13 +1,18 @@
 <?xml version="1.0"?>
 <robot xmlns:xacro="http://www.ros.org/wiki/xacro">
-    <xacro:property name="wheel_mass" value="0.1" />
+    <xacro:property name="rubber_density" value="1100.0" />
     <xacro:property name="wheel_width" value="0.0214" />
     <xacro:property name="wheel_radius" value="0.031755" />
-    <xacro:property name="motor_mass" value="0.333" />
+    <xacro:property name="wheel_mass" value="${rubber_density * pi * wheel_radius * wheel_radius * wheel_width}" />
+    <xacro:property name="motor_mass"  value="0.333" />
+    <xacro:property name="motor_box_x" value="0.06"  />
+    <xacro:property name="motor_box_y" value="0.05"  />
+    <xacro:property name="motor_box_z" value="0.05"  />
     <xacro:macro name="bin_motors" params="prefix">
         <link name="${prefix}left_motor_link">
             <visual>
                 <geometry>
-                    <mesh filename="package://bin_description/meshes/Left Motor.stl" scale="1 1 1"/>
+                    <!-- <mesh filename="package://bin_description/meshes/Left Motor.stl" scale="1 1 1"/> -->
+                    <box size="${motor_box_x} ${motor_box_y} ${motor_box_z}"/>
                 </geometry>
                 <origin xyz="0 0.03 0" rpy="${pi/2} 0 ${-pi/2}"/>
@@ -18,5 +23,6 @@
             <collision>
                 <geometry>
-                    <mesh filename="package://bin_description/meshes/Left Motor.stl" scale="1 1 1"/>
+                    <!-- <mesh filename="package://bin_description/meshes/Left Motor.stl" scale="1 1 1"/> -->
+                    <box size="${motor_box_x} ${motor_box_y} ${motor_box_z}"/>
                 </geometry>
                 <origin xyz="0 0.03 0" rpy="${pi/2} 0 ${-pi/2}"/>
@@ -26,7 +32,7 @@
                 <mass value="${motor_mass}"/>
                 <inertia
-                ixx="9.5017439e-5" ixy="0.0" ixz="0.0"
-                iyy="9.4629109e-5" iyz="-1.779997e-6"
-                izz="4.9374579e-5"/>
+                ixx="${(1/12) * motor_mass * (motor_box_y*motor_box_y + motor_box_z*motor_box_z)}"  ixy="0.0"  ixz="0.0"
+                iyy="${(1/12) * motor_mass * (motor_box_x*motor_box_x + motor_box_z*motor_box_z)}"  iyz="0.0"
+                izz="${(1/12) * motor_mass * (motor_box_x*motor_box_x + motor_box_y*motor_box_y)}"/>
             </inertial>
         </link>
@@ -39,5 +45,6 @@
             <visual>
                 <geometry>
-                    <mesh filename="package://bin_description/meshes/Left Motor.stl" scale="1 1 1"/>
+                    <!-- <mesh filename="package://bin_description/meshes/Left Motor.stl" scale="1 1 1"/> -->
+                    <box size="${motor_box_x} ${motor_box_y} ${motor_box_z}"/>
                 </geometry>
                 <origin xyz="0 -0.03 0" rpy="${pi/2} 0 ${pi/2}"/>
@@ -48,5 +55,6 @@
             <collision>
                 <geometry>
-                    <mesh filename="package://bin_description/meshes/Left Motor.stl" scale="1 1 1"/>
+                    <!-- <mesh filename="package://bin_description/meshes/Left Motor.stl" scale="1 1 1"/> -->
+                    <box size="${motor_box_x} ${motor_box_y} ${motor_box_z}"/>
                 </geometry>
                 <origin xyz="0 -0.03 0" rpy="${pi/2} 0 ${pi/2}"/>
@@ -56,7 +64,7 @@
                 <mass value="${motor_mass}"/>
                 <inertia
-                ixx="9.5017439e-5" ixy="0.0" ixz="0.0"
-                iyy="9.4629109e-5" iyz="-1.779997e-6"
-                izz="4.9374579e-5"/>
+                ixx="${(1/12) * motor_mass * (motor_box_y*motor_box_y + motor_box_z*motor_box_z)}"  ixy="0.0"  ixz="0.0"
+                iyy="${(1/12) * motor_mass * (motor_box_x*motor_box_x + motor_box_z*motor_box_z)}"  iyz="0.0"
+                izz="${(1/12) * motor_mass * (motor_box_x*motor_box_x + motor_box_y*motor_box_y)}"/>
             </inertial>
         </link>
@@ -71,7 +79,8 @@
             <visual>
                 <geometry>
-                    <mesh filename="package://bin_description/meshes/Left Wheel.stl" scale="1 1 1"/>
+                    <!-- <mesh filename="package://bin_description/meshes/Left Wheel.stl" scale="1 1 1"/> -->
+                    <cylinder radius="${wheel_radius}" length="${wheel_width}"/>
                 </geometry>
-                <origin xyz="0 0 0" rpy="0 0 ${pi}"/>
+                <origin xyz="0 0 0" rpy="${pi/2} 0 0"/>
                 <material name="black">
                     <color rgba="0 0 0 1"/>
@@ -80,7 +89,8 @@
             <collision>
                 <geometry>
-                    <mesh filename="package://bin_description/meshes/Left Wheel.stl" scale="1 1 1"/>
+                    <!-- <mesh filename="package://bin_description/meshes/Left Wheel.stl" scale="1 1 1"/> -->
+                    <cylinder radius="${wheel_radius}" length="${wheel_width}"/>
                 </geometry>
-                <origin xyz="0 0 0" rpy="0 0 ${pi}"/>
+                <origin xyz="0 0 0" rpy="${pi/2} 0 0"/>
             </collision>
             <inertial>
@@ -94,7 +104,7 @@
         </link>
         <joint name="${prefix}base_left_wheel_joint" type="continuous">
-            <parent link="${prefix}left_motor_link"/>
+            <parent link="${prefix}base_link"/>
             <child link="${prefix}left_wheel_link"/>
-            <origin xyz="0 0.038 0" rpy="0 0 0"/>
+            <origin xyz="${base_length/4} ${base_width/2 + wheel_width/2} 0" rpy="0 0 0"/>
             <axis xyz="0.0 1.0 0.0"/>
         </joint>
@@ -102,7 +112,8 @@
             <visual>
                 <geometry>
-                    <mesh filename="package://bin_description/meshes/Right Wheel.stl" scale="1 1 1"/>
+                    <!-- <mesh filename="package://bin_description/meshes/Right Wheel.stl" scale="1 1 1"/> -->
+                    <cylinder radius="${wheel_radius}" length="${wheel_width}"/>
                 </geometry>
-                <origin xyz="0 0 0" rpy="0 0 0"/>
+                <origin xyz="0 0 0" rpy="${pi/2} 0 0"/>
                 <material name="black">
                     <color rgba="0 0 0 1"/>
@@ -111,7 +122,8 @@
             <collision>
                 <geometry>
-                    <mesh filename="package://bin_description/meshes/Right Wheel.stl" scale="1 1 1"/>
+                    <!-- <mesh filename="package://bin_description/meshes/Right Wheel.stl" scale="1 1 1"/> -->
+                    <cylinder radius="${wheel_radius}" length="${wheel_width}"/>
                 </geometry>
-                <origin xyz="0 0 0" rpy="0 0 0"/>
+                <origin xyz="0 0 0" rpy="${pi/2} 0 0"/>
             </collision>
             <inertial>
@@ -125,7 +137,7 @@
         </link>
         <joint name="${prefix}base_right_wheel_joint" type="continuous">
-            <parent link="${prefix}right_motor_link"/>
+            <parent link="${prefix}base_link"/>
             <child link="${prefix}right_wheel_link"/>
-            <origin xyz="0 -0.038 0" rpy="0 0 0"/>
+            <origin xyz="${base_length/4} ${-(base_width/2 + wheel_width/2)} 0" rpy="0 0 0"/>
             <axis xyz="0.0 1.0 0.0"/>
         </joint>

File: bin_description/urdf/gazebo/bin_gazebo.urdf.xacro (robot description, xacro)
@@ -33,5 +33,5 @@
                     <range>
                         <min>0.2</min>
-                        <max>30.0</max>
+                        <max>20.0</max>
                         <resolution>0.01</resolution>
                     </range>
@@ -78,12 +78,20 @@
             </sensor>
         </gazebo>
+        <gazebo reference="${prefix}bin_castor_link">
+            <mu1>0.01</mu1>
+            <mu2>0.01</mu2>
+            <kp>100000.0</kp>
+            <kd>10.0</kd>
+            <maxVel>0.01</maxVel>
+            <minDepth>0.001</minDepth>
+        </gazebo>
         <xacro:macro name="wheel_gazebo" params="wheel_name">
             <gazebo reference="${prefix}${wheel_name}_link">
                 <mu1>1.1</mu1>
                 <mu2>1.1</mu2>
-                <kp>1000000.0</kp>
+                <kp>100000.0</kp>
                 <kd>10.0</kd>
                 <minDepth>0.001</minDepth>
-                <maxVel>0.1</maxVel>
+                <maxVel>1.0</maxVel>
                 <fdir1>1 0 0</fdir1>
                 <material>Gazebo/Grey</material>

File: bin_description/urdf/sensors/bin_camera.urdf.xacro (robot description, xacro)
@@ -1,13 +1,15 @@
 <?xml version="1.0"?>
 <robot xmlns:xacro="http://www.ros.org/wiki/xacro">
-    <xacro:property name="camera_mass" value="0.08525" />
+    <xacro:property name="plastic_density" value="1050.0" />
     <xacro:property name="camera_length" value="0.025" />
     <xacro:property name="camera_width" value="0.028062" />
     <xacro:property name="camera_height" value="0.011346" />
+    <xacro:property name="camera_mass" value="${plastic_density * camera_length * camera_width * camera_height}" />
     <xacro:macro name="bin_camera" params="prefix">
         <link name="${prefix}bin_camera_link">
             <visual>
                 <geometry>
-                    <mesh filename="package://bin_description/meshes/camera.stl" scale="1 1 1"/>
+                    <!-- <mesh filename="package://bin_description/meshes/camera.stl" scale="1 1 1"/> -->
+                    <box size="${camera_length} ${camera_width} ${camera_height}"/>
                 </geometry>
                 <origin xyz="0 0 0" rpy="${pi/2} 0 ${pi/2}"/>
@@ -18,5 +20,6 @@
             <collision>
                 <geometry>
-                    <mesh filename="package://bin_description/meshes/camera.stl" scale="1 1 1"/>
+                    <!-- <mesh filename="package://bin_description/meshes/camera.stl" scale="1 1 1"/> -->
+                    <box size="${camera_length} ${camera_width} ${camera_height}"/>
                 </geometry>
                 <origin xyz="0 0 0" rpy="${pi/2} 0 ${pi/2}"/>
@@ -33,5 +36,5 @@
             <parent link="${prefix}bin_top_link"/>
             <child link="${prefix}bin_camera_link"/>
-            <origin xyz="${bin_length/2} 0 0.215" rpy="0 0 0"/>
+            <origin xyz="${bin_length/2 + camera_length/2} 0 ${bin_height/2}" rpy="0 0 0"/>
         </joint>
     </xacro:macro>

File: bin_description/urdf/sensors/bin_lidar.urdf.xacro (robot description, xacro)
@@ -1,7 +1,8 @@
 <?xml version="1.0"?>
 <robot xmlns:xacro="http://www.ros.org/wiki/xacro">
-    <xacro:property name="lidar_mass" value="0.095" />
+    <xacro:property name="plastic_density" value="1050.0" />
     <xacro:property name="lidar_radius" value="0.0175" />
     <xacro:property name="lidar_height" value="0.042" />
+    <xacro:property name="lidar_mass" value="${plastic_density * pi * lidar_radius * lidar_radius * lidar_height}" />
     <xacro:macro name="bin_lidar" params="prefix">
         <link name="${prefix}lidar_link">
@@ -35,5 +36,5 @@
             <child link="${prefix}lidar_link"/>
             <!-- Centred on top face of the cover panel -->
-            <origin xyz="${cover_length/2} 0 ${cover_height / 2 + lidar_height / 2}" rpy="0 0 0"/>
+            <origin xyz="0 0 ${lidar_height/2}" rpy="0 0 0"/>
         </joint>
     </xacro:macro>
