Commit message: Add imu sensor

File: bin_description/urdf/bin_robot.urdf.xacro (robot description, xacro)
@@ -14,4 +14,5 @@
     <xacro:include filename="$(find bin_description)/urdf/ros2_control/bin_ros2_control.xacro"/>
     <xacro:include filename="$(find bin_description)/urdf/gazebo/bin_gazebo.urdf.xacro"/>
+    <xacro:include filename="$(find bin_description)/urdf/sensors/bin_imu.urdf.xacro"/>
     <!-- <xacro:include filename="$(find bin_description)/urdf/sensors/lidar.urdf.xacro"/>
     <xacro:include filename="$(find bin_description)/urdf/body/bin_wheel.urdf.xacro"/>
@@ -38,4 +39,6 @@
     <xacro:bin_camera
       prefix="$(arg prefix)" />
+    <xacro:bin_imu
+    prefix="$(arg prefix)" />
     <!-- <xacro:bin_motors
       prefix="$(arg prefix)"/>
@@ -84,9 +87,4 @@
     <xacro:mecanum_wheel
       prefix="$(arg prefix)"
-      side="back_left"
-      x_reflect="-1"
-      y_reflect="1"/>
-    <xacro:mecanum_wheel
-      prefix="$(arg prefix)"
       side="back_right"
       x_reflect="-1"

File: bin_description/urdf/body/bin_base.urdf.xacro (robot description, xacro)
@@ -3,5 +3,6 @@
 <xacro:property name="base_width" value="0.227" />
 <xacro:property name="base_length" value="0.224725" />
-<xacro:property name="base_height" value="0.140234" />
+<xacro:property name="base_height" value="0.12" />
+<!-- <xacro:property name="base_height" value="0.140234" /> -->
 <xacro:property name="com_x" value="0.00489" />     <!--Center of Mass-->
 <xacro:property name="com_y" value="-0.00007433" />
@@ -18,8 +19,9 @@
         <visual>
             <geometry>
-                <!-- <mesh filename="package://bin_description/meshes/Base.stl" scale="1 1 1"/> -->
-                <box size="${base_length} ${base_width} ${base_height}"/>
+                <mesh filename="package://bin_description/meshes/Base.stl" scale="1 1 1"/>
+                <!-- <box size="${base_length} ${base_width} ${base_height}"/> -->
             </geometry>
-            <origin xyz="0 0 ${base_height/2}" rpy="0 0 0"/>
+            <!-- <origin xyz="0 0 0" rpy="0 0 0"/> -->
+            <origin xyz="-0.01 0 ${base_height}" rpy="0 0 0"/>
             <material name="white">
                 <color rgba="1 1 1 0.5"/>

File: bin_description/urdf/body/bin_cover.urdf.xacro (robot description, xacro)
@@ -10,8 +10,8 @@
             <visual>
                 <geometry>
-                    <!-- <mesh filename="package://bin_description/meshes/Cover.stl" scale="1 1 1"/> -->
-                    <box size="${cover_length} ${cover_width} ${cover_height}"/>
+                    <mesh filename="package://bin_description/meshes/Cover.stl" scale="0.8 0.8 0.8"/>
+                    <!-- <box size="${cover_length} ${cover_width} ${cover_height}"/> -->
                 </geometry>
-                <origin xyz="0.0 0.0 0.0" rpy="0 0 0"/>
+                <origin xyz="${cover_length/2} 0.0 ${-bin_height}" rpy="0 0 0"/>
                 <material name="black">
                     <color rgba="0 0 0 1"/>
@@ -23,5 +23,5 @@
                     <box size="${cover_length} ${cover_width} ${cover_height}"/>
                 </geometry>
-                <origin xyz="0 0 0" rpy="0 0 0"/>
+                <origin xyz="${cover_length/2} 0 0" rpy="0 0 0"/>
             </collision>
             <inertial>
@@ -36,7 +36,7 @@
             <parent link="${prefix}bin_top_link"/>
             <child link="${prefix}bin_cover_link"/>
-            <origin xyz="0 0 ${bin_height}" rpy="0 0 0"/>
+            <origin xyz="${-cover_length/2} 0 ${bin_height}" rpy="0 0 0"/>
             <axis xyz="0 1 0"/>
-            <limit lower="${-pi/2}" upper="0" effort="10" velocity="1.0"/>
+            <limit lower="${-pi/2}" upper="0" effort="100" velocity="1.0"/>
         </joint>
     </xacro:macro>

File: bin_description/urdf/body/bin_top.urdf.xacro (robot description, xacro)
@@ -12,8 +12,9 @@
             <visual>
                 <geometry>
-                    <!-- <mesh filename="package://bin_description/meshes/Bin.stl" scale="1 1 1"/> -->
-                    <box size="${bin_length} ${bin_width} ${bin_height}"/>
+                    <mesh filename="package://bin_description/meshes/Bin.stl" scale="0.8 0.8 0.8"/>
+                    <!-- <box size="${bin_length} ${bin_width} ${bin_height}"/> -->
                 </geometry>
-                <origin xyz="0 0 ${bin_height/2}" rpy="0 0 0"/>
+                <origin xyz="0 0 0" rpy="0 0 0"/>
+                <!-- <origin xyz="0 0 ${bin_height/2}" rpy="0 0 0"/> -->
                 <material name="white">
                     <color rgba="1 1 1 1"/>

File: bin_description/urdf/gazebo/bin_gazebo.urdf.xacro (robot description, xacro)
@@ -86,4 +86,86 @@
             <minDepth>0.001</minDepth>
         </gazebo>
+        <!-- IMU system plugin (required for IMU sensor to publish data) -->
+        <!-- <gazebo>
+            <plugin filename="gz-sim-imu-system" name="gz::sim::systems::Imu"/>
+        </gazebo> -->
+        <!-- IMU SENSOR (MPU 9250 simulation) -->
+        <gazebo reference="${prefix}imu_link">
+            <sensor name="${prefix}imu_sensor" type="imu">
+                <topic>/imu</topic>
+                <update_rate>100</update_rate>
+                <always_on>1</always_on>
+                <visualize>false</visualize>
+                <imu>
+                    <!-- Angular velocity (gyroscope) -->
+                    <angular_velocity>
+                        <x>
+                            <noise type="gaussian">
+                                <mean>0.0</mean>
+                                <stddev>0.009</stddev>
+                                <bias_mean>0.00075</bias_mean>
+                                <bias_stddev>0.005</bias_stddev>
+                                <dynamic_bias_stddev>0.00002</dynamic_bias_stddev>
+                                <dynamic_bias_correlation_time>400.0</dynamic_bias_correlation_time>
+                            </noise>
+                        </x>
+                        <y>
+                            <noise type="gaussian">
+                                <mean>0.0</mean>
+                                <stddev>0.009</stddev>
+                                <bias_mean>0.00075</bias_mean>
+                                <bias_stddev>0.005</bias_stddev>
+                                <dynamic_bias_stddev>0.00002</dynamic_bias_stddev>
+                                <dynamic_bias_correlation_time>400.0</dynamic_bias_correlation_time>
+                            </noise>
+                        </y>
+                        <z>
+                            <noise type="gaussian">
+                                <mean>0.0</mean>
+                                <stddev>0.009</stddev>
+                                <bias_mean>0.00075</bias_mean>
+                                <bias_stddev>0.005</bias_stddev>
+                                <dynamic_bias_stddev>0.00002</dynamic_bias_stddev>
+                                <dynamic_bias_correlation_time>400.0</dynamic_bias_correlation_time>
+                            </noise>
+                        </z>
+                    </angular_velocity>
+                    <!-- Linear acceleration (accelerometer) -->
+                    <linear_acceleration>
+                        <x>
+                            <noise type="gaussian">
+                                <mean>0.0</mean>
+                                <stddev>0.017</stddev>
+                                <bias_mean>0.1</bias_mean>
+                                <bias_stddev>0.001</bias_stddev>
+                                <dynamic_bias_stddev>0.0002</dynamic_bias_stddev>
+                                <dynamic_bias_correlation_time>300.0</dynamic_bias_correlation_time>
+                            </noise>
+                        </x>
+                        <y>
+                            <noise type="gaussian">
+                                <mean>0.0</mean>
+                                <stddev>0.017</stddev>
+                                <bias_mean>0.1</bias_mean>
+                                <bias_stddev>0.001</bias_stddev>
+                                <dynamic_bias_stddev>0.0002</dynamic_bias_stddev>
+                                <dynamic_bias_correlation_time>300.0</dynamic_bias_correlation_time>
+                            </noise>
+                        </y>
+                        <z>
+                            <noise type="gaussian">
+                                <mean>0.0</mean>
+                                <stddev>0.017</stddev>
+                                <bias_mean>0.1</bias_mean>
+                                <bias_stddev>0.001</bias_stddev>
+                                <dynamic_bias_stddev>0.0002</dynamic_bias_stddev>
+                                <dynamic_bias_correlation_time>300.0</dynamic_bias_correlation_time>
+                            </noise>
+                        </z>
+                    </linear_acceleration>
+                </imu>
+                <gz_frame_id>${prefix}imu_link</gz_frame_id>
+            </sensor>
+        </gazebo>
         <xacro:macro name="wheel_gazebo" params="wheel_name">
             <gazebo reference="${prefix}${wheel_name}_link">

File: bin_description/urdf/ros2_control/bin_ros2_control.xacro (robot description, xacro)
@@ -23,4 +23,16 @@
             <xacro:wheel_interfaces name="${prefix}base_right_wheel_joint"/>
             <xacro:wheel_interfaces name="${prefix}base_left_wheel_joint"/>
+            <!-- <sensor name="${prefix}imu_sensor">
+                <state_interface name="orientation.x"/>
+                <state_interface name="orientation.y"/>
+                <state_interface name="orientation.z"/>
+                <state_interface name="orientation.w"/>
+                <state_interface name="angular_velocity.x"/>
+                <state_interface name="angular_velocity.y"/>
+                <state_interface name="angular_velocity.z"/>
+                <state_interface name="linear_acceleration.x"/>
+                <state_interface name="linear_acceleration.y"/>
+                <state_interface name="linear_acceleration.z"/>
+            </sensor> -->
             <joint name="${prefix}bin_cover_joint">
                 <command_interface name="position">

File: bin_description/urdf/sensors/bin_camera.urdf.xacro (robot description, xacro)
@@ -38,4 +38,11 @@
             <origin xyz="${bin_length/2 + camera_length/2} 0 ${bin_height/2}" rpy="0 0 0"/>
         </joint>
+        <!-- Optical/depth frame required by Gazebo gz_frame_id and ROS conventions -->
+        <link name="${prefix}camera_depth_frame"/>
+        <joint name="${prefix}camera_depth_joint" type="fixed">
+            <parent link="${prefix}bin_camera_link"/>
+            <child link="${prefix}camera_depth_frame"/>
+            <origin xyz="0 0 0" rpy="${-pi/2} 0 ${-pi/2}"/>
+        </joint>
     </xacro:macro>
 </robot>
