Commit message: Setup

File: bin_description/urdf/bin_robot.urdf.xacro (robot description, xacro)
@@ -6,4 +6,5 @@
     <xacro:arg name="prefix" default=""/>
     <xacro:arg name="use_gazebo" default="true"/>
+    <xacro:arg name="motor_port" default="/dev/ttyUSB0"/>
     <xacro:include filename="$(find bin_description)/urdf/body/bin_base.urdf.xacro"/>
     <xacro:include filename="$(find bin_description)/urdf/body/bin_wheels.urdf.xacro"/>
@@ -23,5 +24,5 @@
     <!-- <xacro:include filename="$(find bin_description)/urdf/sensors/rgbd_camera.urdf.xacro"/>
     <xacro:include filename="$(find bin_description)/urdf/sensors/imu.urdf.xacro"/> -->
-    <xacro:bin_ros2_control prefix="$(arg prefix)" use_gazebo="$(arg use_gazebo)" />
+    <xacro:bin_ros2_control prefix="$(arg prefix)" use_gazebo="$(arg use_gazebo)" device="$(arg motor_port)" />
     <xacro:bin_gazebo prefix="$(arg prefix)" />
     <xacro:bin_base

File: bin_description/urdf/body/bin_base.urdf.xacro (robot description, xacro)
@@ -15,5 +15,5 @@
 <xacro:property name="castor_mass" value="${metal_density * (4.0/3.0) * pi * castor_radius * castor_radius * castor_radius}" />
 <xacro:macro name="bin_base" params="prefix z_off">
-    <link name="base_footprint"/>
+    <link name="${prefix}base_footprint"/>
     <link name="${prefix}base_link">
         <visual>

File: bin_description/urdf/ros2_control/bin_ros2_control.xacro (robot description, xacro)
@@ -1,5 +1,5 @@
 <?xml version="1.0"?>
 <robot xmlns:xacro="http://www.ros.org/wiki/xacro">
-    <xacro:macro name="bin_ros2_control" params="prefix use_gazebo">
+    <xacro:macro name="bin_ros2_control" params="prefix use_gazebo device:=/dev/ttyUSB0">
         <ros2_control name="BinSystem" type="system">
             <hardware>
@@ -14,5 +14,7 @@
                     <param name="device">/dev/ttyUSB0</param>
                     <param name="baud_rate">57600</param>
-                    <param name="timeout_ms">2000</param>
+                    <!-- Must stay well under the controller_manager cycle budget: this
+                         read blocks the realtime update thread. -->
+                    <param name="timeout_ms">50</param>
                     <param name="enc_counts_per_rev">2475</param>
                     <param name="pid_p_left">10</param>

File: bin_description/urdf/sensors/bin_camera.urdf.xacro (robot description, xacro)
@@ -38,9 +38,16 @@
             <origin xyz="${bin_length/2 + camera_length/2} 0 ${bin_height/2}" rpy="0 0 0"/>
         </joint>
-        <!-- Optical/depth frame required by Gazebo gz_frame_id and ROS conventions -->
-        <link name="${prefix}camera_depth_frame"/>
-        <joint name="${prefix}camera_depth_joint" type="fixed">
+        <!-- Optical frame for the RGB stream. bin_camera_link follows REP-103 body
+             convention (x forward, y left, z up); image data is expressed in REP-105
+             optical convention (z forward along the view axis, x right, y down).
+             The rpy below is that fixed -90/0/-90 rotation and nothing else — do not
+             change it to "fix" an image that looks rotated in RViz.
+             Both camera_ros (frame_id parameter, bin_bringup launch) and the Gazebo
+             sensor (gz_frame_id) must name this frame exactly. Rename in one place
+             and the sim/real parity breaks silently: TF resolves, projections don't. -->
+        <link name="${prefix}camera_rgb_optical_frame"/>
+        <joint name="${prefix}camera_rgb_optical_joint" type="fixed">
             <parent link="${prefix}bin_camera_link"/>
-            <child link="${prefix}camera_depth_frame"/>
+            <child link="${prefix}camera_rgb_optical_frame"/>
             <origin xyz="0 0 0" rpy="${-pi/2} 0 ${-pi/2}"/>
         </joint>
